File: hadi/assignment/opamp-hadi.kicad_pcb (KiCad board)
At the start: 2 copper layers, 20.3 x 12.7 mm, 7 parts, among them U1 LM741

Commit message: Updated version of assignment
Parts:
- added J1: +, Connector_PinHeader_2.00mm:PinHeader_1x02_P2.00mm_Vertical, F.Cu at (127.5, 78.7)
- added J2: SIG, Connector_PinHeader_2.00mm:PinHeader_1x02_P2.00mm_Vertical, F.Cu at (118.3, 78.7)
- renumbered RF to RF1
Connections:
- U1 pad 7: VCC -> Net-(U1-Pad7)
Routing:
- net Net-(U1-Pad7): track 0.00 -> 4.70 mm, vias 0 -> 1
- net Net-(R1-Pad2): track 23.3 -> 27.9 mm, vias 2 -> 4
- net GND: track 19.5 -> 23.2 mm, vias 2 -> 4
Other:
- board size 20.3 x 12.7 mm -> 25.4 x 17.8 mm
- board text added: "-"
- board text added: "GND"
- board text added: "Power Supply"
